File: 1.2/sensor_current.kicad_pcb (KiCad board)
At the start: 2 copper layers, 50 x 50 mm, 19 parts, among them U1 TL084, U2 AD8226

Commit message: error fixed
missing conection detected and eliminated
Connections:
- R2 pad 2: Net-(R2-Pad2) -> /Vref
- R6 pad 2: Net-(R6-Pad2) -> /Vref
Routing:
- net /Vref: track 54.5 -> 66.6 mm, vias 2 -> 3
