File: Wing_CurrentSensor/sensor_current.sch (KiCad schematic (older format))
At the start: 21 parts, among them J1 feather long, J2 feather short, J3 SJ-3524-SMT, U1 TL084, U2 AD8226

Commit message: power at 3.3v and labels update
Connections:
- wire segments 125 -> 126
- no-connect marks 21 -> 22
Changed lines of the file:
@@
 Wire Wire Line
 	3350 3800 3350 4400
-Wire Wire Line
-	3350 4400 3150 4400
-Text Label 3150 4400 2    50   ~ 0
-VBUS
 $Comp
 L Device:CP1 C2
@@
 	3200 2150 3600 2150
 Wire Wire Line
-	3900 1750 3900 1600
-Text Label 3900 1600 0    50   ~ 0
-VBUS
-Wire Wire Line
 	3600 1850 3550 1850
 Wire Wire Line
@@
 Text Notes 1100 650  0    50   ~ 0
 Inputs
-Text Notes 3300 1400 0    50   ~ 0
+Text Notes 3300 1050 0    50   ~ 0
 Instrumentation opamp
 Text Notes 7650 650  0    50   ~ 0
@@
 Text Label 6800 4500 0    50   ~ 0
 VREF
-Text Label 5400 3750 1    50   ~ 0
-VBUS
-Wire Wire Line
-	5400 3950 5400 3750
 $Comp
 L power:GND #PWR0103
@@
 	1    0    0    -1
 $EndComp
+NoConn ~ 10300 4400
+$Comp
+L power:+3.3V #PWR0105
+U 1 1 604C3DB9
+P 5400 3650
+F 0 "#PWR0105" H 5400 3500 50  0001 C CNN
+F 1 "+3.3V" H 5415 3823 50  0000 C CNN
+F 2 "" H 5400 3650 50  0001 C CNN
+F 3 "" H 5400 3650 50  0001 C CNN
+	1    5400 3650
+	1    0    0    -1
+$EndComp
+Wire Wire Line
+	5400 3650 5400 3950
+$Comp
+L power:+3.3V #PWR0106
+U 1 1 604CD61E
+P 3600 4350
+F 0 "#PWR0106" H 3600 4200 50  0001 C CNN
+F 1 "+3.3V" H 3615 4523 50  0000 C CNN
+F 2 "" H 3600 4350 50  0001 C CNN
+F 3 "" H 3600 4350 50  0001 C CNN
+	1    3600 4350
+	1    0    0    -1
+$EndComp
+Wire Wire Line
+	3600 4350 3600 4400
+Wire Wire Line
+	3600 4400 3350 4400
+$Comp
+L power:+3.3V #PWR0107
+U 1 1 604DF341
+P 3900 1350
+F 0 "#PWR0107" H 3900 1200 50  0001 C CNN
+F 1 "+3.3V" H 3915 1523 50  0000 C CNN
+F 2 "" H 3900 1350 50  0001 C CNN
+F 3 "" H 3900 1350 50  0001 C CNN
+	1    3900 1350
+	1    0    0    -1
+$EndComp
+Wire Wire Line
+	3900 1350 3900 1750
 $EndSCHEMATC

Commit message: update connecotr for jumpers
Parts:
- removed JA1, JA2: Conn_01x06, Connector_PinSocket_2.54mm:PinSocket_1x06_P2.54mm_Vertical, symbol Connector_Generic:Conn_01x06
- added J4: Analog Selection, Connector_PinHeader_2.54mm:PinHeader_2x06_P2.54mm_Vertical, symbol Connector_Generic:Conn_02x06_Odd_Even
- C1, C2: symbol Device:CP1 -> sensor_current-rescue:CP1-Device
- D1, D2: symbol pspice:DIODE -> sensor_current-rescue:DIODE-pspice
- J1: symbol Connector_Generic:Conn_01x16 -> sensor_current-rescue:Conn_01x16-Connector_Generic
- J2: symbol Connector_Generic:Conn_01x12 -> sensor_current-rescue:Conn_01x12-Connector_Generic
- J3: symbol jack:SJ-3524-SMT -> sensor_current-rescue:SJ-3524-SMT-jack
- R1, R2, R3, R4, R5, R6, R7, R8, R9: symbol Device:R -> sensor_current-rescue:R-Device
- RV1: symbol Device:R_POT -> sensor_current-rescue:R_POT-Device
- U1: symbol Amplifier_Operational:TL084 -> sensor_current-rescue:TL084-Amplifier_Operational
- U2: symbol Amplifier_Instrumentation:AD8421 -> sensor_current-rescue:AD8421-Amplifier_Instrumentation
Changed lines of the file:
@@
 	3350 3800 3350 4400
 $Comp
-L Device:CP1 C2
+L sensor_current-rescue:CP1-Device C2
 U 1 1 601E5B1F
 P 3350 4950
@@
 $EndComp
 $Comp
-L Amplifier_Operational:TL084 U1
+L sensor_current-rescue:TL084-Amplifier_Operational U1
 U 5 1 601E5B25
 P 3050 3900
@@
 $EndComp
 $Comp
-L power:GND #PWR0102
+L sensor_current-rescue:GND-power #PWR0102
 U 1 1 60295F05
 P 3350 5500
@@
 	7200 2150 7100 2150
 $Comp
-L Device:R R2
+L sensor_current-rescue:R-Device R2
 U 1 1 602E05A9
 P 7100 2350
@@
 	9050 2200 9050 2150
 $Comp
-L Device:R R6
+L sensor_current-rescue:R-Device R6
 U 1 1 602E8C25
 P 9050 2350
@@
 	9200 1450 9050 1450
 $Comp
-L Device:R R7
+L sensor_current-rescue:R-Device R7
 U 1 1 602F1EB7
 P 9350 1450
@@
 	9200 1200 9050 1200
 $Comp
-L Device:CP1 C1
+L sensor_current-rescue:CP1-Device C1
 U 1 1 602F1EBF
 P 9350 1200
@@
 	6500 1200 7600 1200
 $Comp
-L Device:R R4
+L sensor_current-rescue:R-Device R4
 U 1 1 602F1EC9
 P 7750 1200
@@
 	8600 1450 8350 1450
 $Comp
-L Device:R R5
+L sensor_current-rescue:R-Device R5
 U 1 1 602F1ED1
 P 8750 1450
@@
 	7050 1550 7250 1550
 $Comp
-L Device:R R3
+L sensor_current-rescue:R-Device R3
 U 1 1 602F1EE8
 P 7650 1450
@@
 	6950 1550 7050 1550
 $Comp
-L pspice:DIODE D1
+L sensor_current-rescue:DIODE-pspice D1
 U 1 1 602F1EFE
 P 8050 1750
@@
 $EndComp
 $Comp
-L Device:R R1
+L sensor_current-rescue:R-Device R1
 U 1 1 602F1F0A
 P 6800 1550
@@
 	8250 5950 8250 3200
 $Comp
-L Device:R R8
+L sensor_current-rescue:R-Device R8
 U 1 1 60371C97
 P 5400 4100
@@
 $EndComp
 $Comp
-L Device:R R9
+L sensor_current-rescue:R-Device R9
 U 1 1 60372648
 P 5400 4600
@@
 $EndComp
 $Comp
-L power:GND #PWR0101
+L sensor_current-rescue:GND-power #PWR0101
 U 1 1 6037A08F
 P 5400 4950
@@
 VREF
 $Comp
-L power:GND #PWR0103
+L sensor_current-rescue:GND-power #PWR0103
 U 1 1 603897CB
 P 3900 2550
@@
 	3350 5100 3350 5500
 $Comp
-L power:GND #PWR0104
+L sensor_current-rescue:GND-power #PWR0104
 U 1 1 603A380E
 P 2550 4600
@@
 	2550 3800 2550 4600
 $Comp
-L Amplifier_Operational:TL084 U1
+L sensor_current-rescue:TL084-Amplifier_Operational U1
 U 4 1 60375049
 P 6250 4500
@@
 	5400 4400 5400 4450
 $Comp
-L Amplifier_Operational:TL084 U1
+L sensor_current-rescue:TL084-Amplifier_Operational U1
 U 2 1 602E8C1B
 P 9450 2050
@@
 $EndComp
 $Comp
-L Amplifier_Operational:TL084 U1
+L sensor_current-rescue:TL084-Amplifier_Operational U1
 U 1 1 602E05B2
 P 7500 2050
@@
 	9050 2750 9150 2750
 $Comp
-L Connector_Generic:Conn_01x16 J1
+L sensor_current-rescue:Conn_01x16-Connector_Generic J1
 U 1 1 5D375C76
 P 9450 4600
@@
 $EndComp
 $Comp
-L Connector_Generic:Conn_01x12 J2
+L sensor_current-rescue:Conn_01x12-Connector_Generic J2
 U 1 1 5D375CC4
 P 9850 4800
@@
 	10050 5300 10300 5300
 $Comp
-L power:+3.3V #PWR01
+L sensor_current-rescue:+3.3V-power #PWR01
 U 1 1 5D37877D
 P 8900 3800
@@
 $EndComp
 $Comp
-L power:GND #PWR02
+L sensor_current-rescue:GND-power #PWR02
 U 1 1 5D3787E4
 P 8400 4200
@@
 	9050 4200 9250 4200
 $Comp
-L jack:SJ-3524-SMT J3
+L sensor_current-rescue:SJ-3524-SMT-jack J3
 U 1 1 6040A716
 P 1000 1900
@@
 	4100 2350 4300 2350
 $Comp
-L Amplifier_Instrumentation:AD8421 U2
+L sensor_current-rescue:AD8421-Amplifier_Instrumentation U2
 U 1 1 602A5CCD
 P 4000 2050
@@
 Wire Wire Line
 	9800 1900 9800 1800
-$Comp
-L Connector_Generic:Conn_01x06 JA2
-U 1 1 60472DE0
-P 10250 1700
-F 0 "JA2" H 10330 1692 50  0000 L CNN
-F 1 "Conn_01x06" H 10330 1601 50  0000 L CNN
-F 2 "Connector_PinSocket_2.54mm:PinSocket_1x06_P2.54mm_Vertical" H 10250 1700 50  0001 C CNN
-F 3 "~" H 10250 1700 50  0001 C CNN
-	1    10250 1700
-	1    0    0    -1
-$EndComp
-$Comp
-L Connector_Generic:Conn_01x06 JA1
-U 1 1 60473370
-P 1250 4300
-F 0 "JA1" H 1330 4292 50  0000 L CNN
-F 1 "Conn_01x06" H 1330 4201 50  0000 L CNN
-F 2 "Connector_PinSocket_2.54mm:PinSocket_1x06_P2.54mm_Vertical" H 1250 4300 50  0001 C CNN
-F 3 "~" H 1250 4300 50  0001 C CNN
-	1    1250 4300
-	-1   0    0    1
-$EndComp
 Wire Wire Line
 	9800 1500 10050 1500
@@
 Wire Wire Line
 	9800 1950 9800 1900
-Text Label 1550 4000 0    50   ~ 0
+Text Label 10650 2000 0    50   ~ 0
 A0
-Text Label 1550 4100 0    50   ~ 0
+Text Label 10650 1900 0    50   ~ 0
 A1
-Text Label 1550 4200 0    50   ~ 0
+Text Label 10650 1800 0    50   ~ 0
 A2
-Text Label 1550 4300 0    50   ~ 0
+Text Label 10650 1700 0    50   ~ 0
 A3
-Text Label 1550 4400 0    50   ~ 0
+Text Label 10650 1600 0    50   ~ 0
 A4
-Text Label 1550 4500 0    50   ~ 0
+Text Label 10650 1500 0    50   ~ 0
 A5
 Wire Wire Line
-	1450 4000 1550 4000
-Wire Wire Line
-	1450 4100 1550 4100
-Wire Wire Line
-	1450 4200 1550 4200
-Wire Wire Line
-	1450 4300 1550 4300
-Wire Wire Line
-	1450 4400 1550 4400
-Wire Wire Line
-	1450 4500 1550 4500
+	10550 2000 10650 2000
+Wire Wire Line
+	10550 1900 10650 1900
+Wire Wire Line
+	10550 1800 10650 1800
+Wire Wire Line
+	10550 1700 10650 1700
+Wire Wire Line
+	10550 1600 10650 1600
+Wire Wire Line
+	10550 1500 10650 1500
 Wire Notes Line
 	1950 3150 1950 5950
 $Comp
-L pspice:DIODE D2
+L sensor_current-rescue:DIODE-pspice D2
 U 1 1 602F1EF8
 P 8350 1750
@@
 $EndComp
 $Comp
-L Device:R_POT RV1
+L sensor_current-rescue:R_POT-Device RV1
 U 1 1 602A5CBE
 P 3200 2000
@@
 NoConn ~ 10300 4400
 $Comp
-L power:+3.3V #PWR0105
+L sensor_current-rescue:+3.3V-power #PWR0105
 U 1 1 604C3DB9
 P 5400 3650
@@
 	5400 3650 5400 3950
 $Comp
-L power:+3.3V #PWR0106
+L sensor_current-rescue:+3.3V-power #PWR0106
 U 1 1 604CD61E
 P 3600 4350
@@
 	3600 4400 3350 4400
 $Comp
-L power:+3.3V #PWR0107
+L sensor_current-rescue:+3.3V-power #PWR0107
 U 1 1 604DF341
 P 3900 1350
@@
 Wire Wire Line
 	3900 1350 3900 1750
+$Comp
+L Connector_Generic:Conn_02x06_Odd_Even J4
+U 1 1 604C74A8
+P 10250 1700
+F 0 "J4" H 10300 2117 50  0000 C CNN
+F 1 "Analog Selection" H 10300 2026 50  0000 C CNN
+F 2 "Connector_PinHeader_2.54mm:PinHeader_2x06_P2.54mm_Vertical" H 10250 1700 50  0001 C CNN
+F 3 "~" H 10250 1700 50  0001 C CNN
+	1    10250 1700
+	1    0    0    -1
+$EndComp
 $EndSCHEMATC

Commit message: Add_Connector
Connections:
- net GND: now also J3.1, U2.1 (-)
- net IN+: now also J3.3
- net IN-: no longer names the net of J3.2
- net IN-: no longer U2.1 (-)
- no-connect marks 22 -> 21
Changed lines of the file:
@@
 Wire Wire Line
 	8400 4100 9250 4100
-Text Label 1650 2000 0    50   ~ 0
+Text Label 1650 1900 0    50   ~ 0
 IN+
-Text Label 1700 1800 0    50   ~ 0
+Text Label 1700 1700 0    50   ~ 0
 IN-
 NoConn ~ 10050 5000
@@
 $EndComp
 Wire Wire Line
-	1500 1800 1700 1800
-Wire Wire Line
-	1500 2000 1650 2000
+	1500 1700 1595 1700
+Wire Wire Line
+	1500 1900 1650 1900
 NoConn ~ 10300 4900
 NoConn ~ 10300 4800
@@
 	1    0    0    -1
 $EndComp
-NoConn ~ 1500 1900
-NoConn ~ 1500 1700
+NoConn ~ 1500 1800
 NoConn ~ 9050 4800
 NoConn ~ 9050 4900
@@
 	1    0    0    -1
 $EndComp
+$Comp
+L power:GND #PWR0108
+U 1 1 60D403E1
+P 1595 1740
+F 0 "#PWR0108" H 1595 1490 50  0001 C CNN
+F 1 "GND" H 1600 1567 50  0000 C CNN
+F 2 "" H 1595 1740 50  0001 C CNN
+F 3 "" H 1595 1740 50  0001 C CNN
+	1    1595 1740
+	1    0    0    -1
+$EndComp
+Wire Wire Line
+	1595 1740 1595 1700
+Connection ~ 1595 1700
+Wire Wire Line
+	1595 1700 1700 1700
 $EndSCHEMATC

Commit message: Change_BOM
Parts:
- J3: value SJ-3524-SMT -> PJ-320B
Changed lines of the file:
@@
 P 1000 1900
 F 0 "J3" H 1107 2367 50  0000 C CNN
-F 1 "SJ-3524-SMT" H 1107 2276 50  0000 C CNN
+F 1 "PJ-320B" H 1107 2276 50  0000 C CNN
 F 2 "CUI_SJ-3524-SMT" H 1000 1900 50  0001 L BNN
 F 3 "" H 1000 1900 50  0001 L BNN
