File: Wing_CurrentSensor/sensor_current.sch (KiCad schematic (older format))
At the start: 25 parts, among them J1 feather long, J2 feather short, J3 PJ-320B, U1 MCP6009, U2 AD8226

Commit message: Init_BOM_Change3D_Model
Parts:
- C1: #LCSC (none) -> C326057
- C2: #LCSC (none) -> C360619
- D1, D2: #LCSC (none) -> C305438; #Mouser (none) -> 512-1N4148WS
- J3: footprint CUI_SJ-3524-SMT -> PJ-313D-6A; #LCSC (none) -> C95463
- R1, R3, R4, R7, R8, R9: #LCSC (none) -> C115295
- U1: #Mouser (none) -> 579-MCP6009-E/SL
- U2: #Mouser (none) -> 584-AD8226ARZ
Changed lines of the file:
@@
 F 2 "Capacitor_SMD:C_0805_2012Metric_Pad1.18x1.45mm_HandSolder" H 3350 4950 50  0001 C CNN
 F 3 "~" H 3350 4950 50  0001 C CNN
+F 4 "C360619" H 3350 4950 50  0001 C CNN "#LCSC"
 	1    3350 4950
 	1    0    0    -1
@@
 F 2 "Package_SO:SO-14_3.9x8.65mm_P1.27mm" H 3000 4000 50  0001 C CNN
 F 3 "http://www.ti.com/lit/ds/symlink/tl081.pdf" H 3100 4100 50  0001 C CNN
+F 4 "579-MCP6009-E/SL" H 3050 3900 50  0001 C CNN "#Mouser"
 	5    3050 3900
 	0    1    1    0
@@
 F 2 "Resistor_SMD:R_0805_2012Metric_Pad1.20x1.40mm_HandSolder" V 9280 1450 50  0001 C CNN
 F 3 "~" H 9350 1450 50  0001 C CNN
+F 4 "C115295" H 9350 1450 50  0001 C CNN "#LCSC"
 	1    9350 1450
 	0    1    1    0
@@
 F 2 "Capacitor_SMD:C_0805_2012Metric_Pad1.18x1.45mm_HandSolder" H 9350 1200 50  0001 C CNN
 F 3 "~" H 9350 1200 50  0001 C CNN
+F 4 "C326057" H 9350 1200 50  0001 C CNN "#LCSC"
 	1    9350 1200
 	0    1    1    0
@@
 F 2 "Resistor_SMD:R_0805_2012Metric_Pad1.20x1.40mm_HandSolder" V 7680 1200 50  0001 C CNN
 F 3 "~" H 7750 1200 50  0001 C CNN
+F 4 "C115295" H 7750 1200 50  0001 C CNN "#LCSC"
 	1    7750 1200
 	0    -1   -1   0
@@
 F 2 "Resistor_SMD:R_0805_2012Metric_Pad1.20x1.40mm_HandSolder" V 7580 1445 50  0001 C CNN
 F 3 "~" H 7650 1445 50  0001 C CNN
+F 4 "C115295" H 7650 1445 50  0001 C CNN "#LCSC"
 	1    7650 1445
 	0    -1   -1   0
@@
 F 2 "Diode_SMD:D_SOD-323F" H 8050 1795 50  0001 C CNN
 F 3 "~" H 8050 1795 50  0001 C CNN
+F 4 "C305438" H 8050 1795 50  0001 C CNN "#LCSC"
+F 5 "512-1N4148WS" H 8050 1795 50  0001 C CNN "#Mouser"
 	1    8050 1795
 	0    -1   -1   0
@@
 F 2 "Resistor_SMD:R_0805_2012Metric_Pad1.20x1.40mm_HandSolder" V 6730 1445 50  0001 C CNN
 F 3 "~" H 6800 1445 50  0001 C CNN
+F 4 "C115295" H 6800 1445 50  0001 C CNN "#LCSC"
 	1    6800 1445
 	0    -1   -1   0
@@
 F 2 "Resistor_SMD:R_0805_2012Metric_Pad1.20x1.40mm_HandSolder" V 5330 4100 50  0001 C CNN
 F 3 "~" H 5400 4100 50  0001 C CNN
+F 4 "C115295" H 5400 4100 50  0001 C CNN "#LCSC"
 	1    5400 4100
 	1    0    0    -1
@@
 F 2 "Resistor_SMD:R_0805_2012Metric_Pad1.20x1.40mm_HandSolder" V 5330 4600 50  0001 C CNN
 F 3 "~" H 5400 4600 50  0001 C CNN
+F 4 "C115295" H 5400 4600 50  0001 C CNN "#LCSC"
 	1    5400 4600
 	1    0    0    -1
@@
 F 2 "Package_SO:SO-14_3.9x8.65mm_P1.27mm" H 6200 4600 50  0001 C CNN
 F 3 "http://www.ti.com/lit/ds/symlink/tl081.pdf" H 6300 4700 50  0001 C CNN
+F 4 "579-MCP6009-E/SL" H 6250 4500 50  0001 C CNN "#Mouser"
 	4    6250 4500
 	1    0    0    -1
@@
 F 2 "Package_SO:SO-14_3.9x8.65mm_P1.27mm" H 9400 2150 50  0001 C CNN
 F 3 "http://www.ti.com/lit/ds/symlink/tl081.pdf" H 9500 2250 50  0001 C CNN
+F 4 "579-MCP6009-E/SL" H 9450 2050 50  0001 C CNN "#Mouser"
 	2    9450 2050
 	1    0    0    1
@@
 F 2 "Package_SO:SO-14_3.9x8.65mm_P1.27mm" H 7450 2150 50  0001 C CNN
 F 3 "http://www.ti.com/lit/ds/symlink/tl081.pdf" H 7550 2250 50  0001 C CNN
+F 4 "579-MCP6009-E/SL" H 7500 2050 50  0001 C CNN "#Mouser"
 	1    7500 2050
 	1    0    0    1
@@
 F 0 "J3" H 1107 2367 50  0000 C CNN
 F 1 "PJ-320B" H 1107 2276 50  0000 C CNN
-F 2 "CUI_SJ-3524-SMT" H 1000 1900 50  0001 L BNN
+F 2 "PJ-313D-6A" H 1000 1900 50  0001 L BNN
 F 3 "" H 1000 1900 50  0001 L BNN
 F 4 "CUI Inc" H 1000 1900 50  0001 L BNN "MF"
 F 5 "1.03" H 1000 1900 50  0001 L BNN "PARTREV"
 F 6 "Manufacturer recommendations" H 1000 1900 50  0001 L BNN "STANDARD"
+F 7 "C95463" H 1000 1900 50  0001 C CNN "#LCSC"
 	1    1000 1900
 	1    0    0    -1
@@
 F 2 "Package_SO:SOIC-8_3.9x4.9mm_P1.27mm" H 3700 2050 50  0001 C CNN
 F 3 "https://www.analog.com/media/en/technical-documentation/data-sheets/AD8421.pdf" H 4350 1650 50  0001 C CNN
+F 4 "584-AD8226ARZ" H 4000 2050 50  0001 C CNN "#Mouser"
 	1    4000 2050
 	1    0    0    -1
@@
 F 2 "Diode_SMD:D_SOD-323F" H 8350 1750 50  0001 C CNN
 F 3 "~" H 8350 1750 50  0001 C CNN
+F 4 "C305438" H 8350 1750 50  0001 C CNN "#LCSC"
+F 5 "512-1N4148WS" H 8350 1750 50  0001 C CNN "#Mouser"
 	1    8350 1750
 	0    1    1    0

Commit message: Finish_BOM
Parts:
- R2, R5: #LCSC (none) -> C332873
- R6: #LCSC (none) -> C139892
Changed lines of the file:
@@
 F 1 "0.1μ " V 3189 4950 50  0000 C CNN
 F 2 "Capacitor_SMD:C_0805_2012Metric_Pad1.18x1.45mm_HandSolder" H 3350 4950 50  0001 C CNN
-F 3 "~" H 3350 4950 50  0001 C CNN
+F 3 "https://datasheet.lcsc.com/lcsc/1912111437_CCTC-TCC0805X7R104M500DT_C360619.pdf" H 3350 4950 50  0001 C CNN
 F 4 "C360619" H 3350 4950 50  0001 C CNN "#LCSC"
 	1    3350 4950
@@
 F 1 "5K" H 7170 2305 50  0000 L CNN
 F 2 "Resistor_SMD:R_0805_2012Metric_Pad1.20x1.40mm_HandSolder" V 7030 2350 50  0001 C CNN
-F 3 "~" H 7100 2350 50  0001 C CNN
+F 3 "https://datasheet.lcsc.com/lcsc/1912111437_RALEC-RTT055001FTP_C332873.pdf" H 7100 2350 50  0001 C CNN
+F 4 "C332873" H 7100 2350 50  0001 C CNN "#LCSC"
 	1    7100 2350
 	1    0    0    -1
@@
 F 1 "3.3K" H 9120 2305 50  0000 L CNN
 F 2 "Resistor_SMD:R_0805_2012Metric_Pad1.20x1.40mm_HandSolder" V 8980 2350 50  0001 C CNN
-F 3 "~" H 9050 2350 50  0001 C CNN
+F 3 "https://datasheet.lcsc.com/lcsc/1811061712_FH-Guangdong-Fenghua-Advanced-Tech-RS-05K332JT_C139892.pdf" H 9050 2350 50  0001 C CNN
+F 4 "C139892" H 9050 2350 50  0001 C CNN "#LCSC"
 	1    9050 2350
 	1    0    0    -1
@@
 F 1 "10K" H 9420 1405 50  0000 L CNN
 F 2 "Resistor_SMD:R_0805_2012Metric_Pad1.20x1.40mm_HandSolder" V 9280 1450 50  0001 C CNN
-F 3 "~" H 9350 1450 50  0001 C CNN
+F 3 "https://datasheet.lcsc.com/lcsc/1811141124_FH-Guangdong-Fenghua-Advanced-Tech-RS-05K103JT_C115295.pdf" H 9350 1450 50  0001 C CNN
 F 4 "C115295" H 9350 1450 50  0001 C CNN "#LCSC"
 	1    9350 1450
@@
 F 1 "10 μ " V 9189 1200 50  0000 C CNN
 F 2 "Capacitor_SMD:C_0805_2012Metric_Pad1.18x1.45mm_HandSolder" H 9350 1200 50  0001 C CNN
-F 3 "~" H 9350 1200 50  0001 C CNN
+F 3 "https://datasheet.lcsc.com/lcsc/1811031143_YAGEO-CC0603KRX5R6BB106_C326057.pdf" H 9350 1200 50  0001 C CNN
 F 4 "C326057" H 9350 1200 50  0001 C CNN "#LCSC"
 	1    9350 1200
@@
 F 1 "10K" H 7820 1155 50  0000 L CNN
 F 2 "Resistor_SMD:R_0805_2012Metric_Pad1.20x1.40mm_HandSolder" V 7680 1200 50  0001 C CNN
-F 3 "~" H 7750 1200 50  0001 C CNN
+F 3 "https://datasheet.lcsc.com/lcsc/1811141124_FH-Guangdong-Fenghua-Advanced-Tech-RS-05K103JT_C115295.pdf" H 7750 1200 50  0001 C CNN
 F 4 "C115295" H 7750 1200 50  0001 C CNN "#LCSC"
 	1    7750 1200
@@
 F 1 "5K" H 8820 1405 50  0000 L CNN
 F 2 "Resistor_SMD:R_0805_2012Metric_Pad1.20x1.40mm_HandSolder" V 8680 1450 50  0001 C CNN
-F 3 "~" H 8750 1450 50  0001 C CNN
+F 3 "https://datasheet.lcsc.com/lcsc/1912111437_RALEC-RTT055001FTP_C332873.pdf" H 8750 1450 50  0001 C CNN
+F 4 "C332873" H 8750 1450 50  0001 C CNN "#LCSC"
 	1    8750 1450
 	0    -1   -1   0
@@
 F 1 "10K" H 7720 1400 50  0000 L CNN
 F 2 "Resistor_SMD:R_0805_2012Metric_Pad1.20x1.40mm_HandSolder" V 7580 1445 50  0001 C CNN
-F 3 "~" H 7650 1445 50  0001 C CNN
+F 3 "https://datasheet.lcsc.com/lcsc/1811141124_FH-Guangdong-Fenghua-Advanced-Tech-RS-05K103JT_C115295.pdf" H 7650 1445 50  0001 C CNN
 F 4 "C115295" H 7650 1445 50  0001 C CNN "#LCSC"
 	1    7650 1445
@@
 F 1 "1N4148WS" V 7930 1890 50  0000 L CNN
 F 2 "Diode_SMD:D_SOD-323F" H 8050 1795 50  0001 C CNN
-F 3 "~" H 8050 1795 50  0001 C CNN
+F 3 "https://datasheet.lcsc.com/lcsc/1810201910_Foshan-Blue-Rocket-Elec-1N4148WS_C305438.pdf" H 8050 1795 50  0001 C CNN
 F 4 "C305438" H 8050 1795 50  0001 C CNN "#LCSC"
 F 5 "512-1N4148WS" H 8050 1795 50  0001 C CNN "#Mouser"
@@
 F 1 "10K" H 6870 1400 50  0000 L CNN
 F 2 "Resistor_SMD:R_0805_2012Metric_Pad1.20x1.40mm_HandSolder" V 6730 1445 50  0001 C CNN
-F 3 "~" H 6800 1445 50  0001 C CNN
+F 3 "https://datasheet.lcsc.com/lcsc/1811141124_FH-Guangdong-Fenghua-Advanced-Tech-RS-05K103JT_C115295.pdf" H 6800 1445 50  0001 C CNN
 F 4 "C115295" H 6800 1445 50  0001 C CNN "#LCSC"
 	1    6800 1445
@@
 F 1 "10K" H 5470 4055 50  0000 L CNN
 F 2 "Resistor_SMD:R_0805_2012Metric_Pad1.20x1.40mm_HandSolder" V 5330 4100 50  0001 C CNN
-F 3 "~" H 5400 4100 50  0001 C CNN
+F 3 "https://datasheet.lcsc.com/lcsc/1811141124_FH-Guangdong-Fenghua-Advanced-Tech-RS-05K103JT_C115295.pdf" H 5400 4100 50  0001 C CNN
 F 4 "C115295" H 5400 4100 50  0001 C CNN "#LCSC"
 	1    5400 4100
@@
 F 1 "10K" H 5470 4555 50  0000 L CNN
 F 2 "Resistor_SMD:R_0805_2012Metric_Pad1.20x1.40mm_HandSolder" V 5330 4600 50  0001 C CNN
-F 3 "~" H 5400 4600 50  0001 C CNN
+F 3 "https://datasheet.lcsc.com/lcsc/1811141124_FH-Guangdong-Fenghua-Advanced-Tech-RS-05K103JT_C115295.pdf" H 5400 4600 50  0001 C CNN
 F 4 "C115295" H 5400 4600 50  0001 C CNN "#LCSC"
 	1    5400 4600
@@
 F 1 "PJ-320B" H 1107 2276 50  0000 C CNN
 F 2 "PJ-313D-6A" H 1000 1900 50  0001 L BNN
-F 3 "" H 1000 1900 50  0001 L BNN
+F 3 "https://datasheet.lcsc.com/lcsc/1810141713_Korean-Hroparts-Elec-PJ-313D-6A_C95463.pdf" H 1000 1900 50  0001 L BNN
 F 4 "CUI Inc" H 1000 1900 50  0001 L BNN "MF"
 F 5 "1.03" H 1000 1900 50  0001 L BNN "PARTREV"
@@
 F 1 "1N4148WS" V 8395 1878 50  0000 L CNN
 F 2 "Diode_SMD:D_SOD-323F" H 8350 1750 50  0001 C CNN
-F 3 "~" H 8350 1750 50  0001 C CNN
+F 3 "https://datasheet.lcsc.com/lcsc/1810201910_Foshan-Blue-Rocket-Elec-1N4148WS_C305438.pdf" H 8350 1750 50  0001 C CNN
 F 4 "C305438" H 8350 1750 50  0001 C CNN "#LCSC"
 F 5 "512-1N4148WS" H 8350 1750 50  0001 C CNN "#Mouser"
